Commit message: Add camera and material to to the robot

File: udacity_bot/urdf/udacity_bot.xacro (robot description, xacro)
@@ -1,4 +1,5 @@
 <?xml version='1.0'?>
 <robot name="udacity_bot" xmlns:xacro="http://www.ros.org/wiki/xacro">
+  <xacro:include filename="$(find udacity_bot)/urdf/udacity_bot.gazebo" />
   <link name="robot_footprint"></link>
   <joint name="robot_footprint_joint" type="fixed">
@@ -24,5 +25,5 @@
       </geometry>
     </collision>
-    <visual name='chassis_visual'>
+    <visual>
       <origin xyz="0 0 0" rpy=" 0 0 0"/>
       <geometry>
@@ -36,5 +37,5 @@
       </geometry>
     </collision>
-    <visual name='back_caster_visual'>
+    <visual>
       <origin xyz="-0.15 0 -0.05" rpy=" 0 0 0"/>
       <geometry>
@@ -48,5 +49,5 @@
       </geometry>
     </collision>
-    <visual name='front_caster_visual'>
+    <visual>
       <origin xyz="0.15 0 -0.05" rpy=" 0 0 0"/>
       <geometry>
@@ -56,5 +57,4 @@
   </link>
   <link name='left_wheel'>
-    <!-- <pose>0 0 0.1 0 0 0</pose> -->
     <inertial>
       <mass value="5.0"/>
@@ -72,5 +72,5 @@
       </geometry>
     </collision>
-    <visual name='chassis_visual'>
+    <visual>
       <origin xyz="0 0 0" rpy="0 1.5707 1.5707"/>
       <geometry>
@@ -88,5 +88,4 @@
   </joint>
   <link name='right_wheel'>
-    <!-- <pose>0 0 0.1 0 0 0</pose> -->
     <inertial>
       <mass value="5.0"/>
@@ -104,5 +103,5 @@
       </geometry>
     </collision>
-    <visual name='chassis_visual'>
+    <visual>
       <origin xyz="0 0 0" rpy="0 1.5707 1.5707"/>
       <geometry>
@@ -119,3 +118,63 @@
     <dynamics damping="1.0" friction="1.0" />
   </joint>
+  <link name='camera'>
+    <inertial>
+      <mass value="0.1"/>
+      <origin xyz="0 0 0" rpy="0 0 0"/>
+      <inertia ixx="1e-6" ixy="0" ixz="0" iyy="1e-6" iyz="0" izz="1e-6" />
+    </inertial>
+    <collision name='collision'>
+      <origin xyz="0 0 0" rpy="0 0 0"/>
+      <geometry>
+        <box size="0.05 0.05 0.05" />
+      </geometry>
+    </collision>
+    <visual>
+      <origin xyz="0 0 0" rpy="0 0 0"/>
+      <geometry>
+        <box size="0.05 0.05 0.05" />
+      </geometry>
+    </visual>
+  </link>
+  <joint name="camera_joint" type="fixed">
+    <origin xyz="0.2 0 0" rpy="0 0 0" />
+    <parent link="chassis" />
+    <child link="camera" />
+  </joint>
+  <link name='hokuyo'>
+    <inertial>
+      <mass value="0.1"/>
+      <origin xyz="0 0 0" rpy="0 0 0"/>
+      <inertia ixx="1e-6" ixy="0" ixz="0" iyy="1e-6" iyz="0" izz="1e-6" />
+    </inertial>
+    <collision name='collision'>
+      <origin xyz="0 0 0" rpy="0 0 0"/>
+      <geometry>
+        <box size="0.1 0.1 0.1" />
+      </geometry>
+    </collision>
+    <visual>
+      <origin xyz="0 0 0" rpy="0 0 0"/>
+      <geometry>
+        <mesh filename="package://udacity_bot/meshes/hokuyo.dae" />
+      </geometry>
+    </visual>
+  </link>
+  <joint name="hokuyo_joint" type="fixed">
+    <origin xyz="0.15 0 0.1" rpy="0 0 0" />
+    <parent link="chassis" />
+    <child link="hokuyo" />
+  </joint>
+  <gazebo reference="chassis">
+    <material>Gazebo/Blue</material>
+  </gazebo>
+  <gazebo reference="left_wheel">
+    <material>Gazebo/Green</material>
+  </gazebo>
+  <gazebo reference="right_wheel">
+    <material>Gazebo/Green</material>
+  </gazebo>
+  <gazebo reference="camera">
+    <material>Gazebo/Red</material>
+  </gazebo>
 </robot>
