Commit message: Continue rename of package to slam_bot.\nConfigure RGB-D camera

File: slam_bot/urdf/slam_bot.xacro (robot description, xacro)
@@ -1,5 +1,5 @@
 <?xml version='1.0'?>
-<robot name="udacity_bot" xmlns:xacro="http://www.ros.org/wiki/xacro">
-  <xacro:include filename="$(find udacity_bot)/urdf/udacity_bot.gazebo" />
+<robot name="slam_bot" xmlns:xacro="http://www.ros.org/wiki/xacro">
+  <xacro:include filename="$(find slam_bot)/urdf/slam_bot.gazebo" />
   <link name="robot_footprint"></link>
   <joint name="robot_footprint_joint" type="fixed">
@@ -118,5 +118,5 @@
     <dynamics damping="1.0" friction="1.0" />
   </joint>
-  <link name='camera'>
+  <link name="camera">
     <inertial>
       <mass value="0.1"/>
@@ -124,5 +124,5 @@
       <inertia ixx="1e-6" ixy="0" ixz="0" iyy="1e-6" iyz="0" izz="1e-6" />
     </inertial>
-    <collision name='collision'>
+    <collision name="collision">
       <origin xyz="0 0 0" rpy="0 0 0"/>
       <geometry>
@@ -142,4 +142,10 @@
     <child link="camera" />
   </joint>
+  <link name="camera_rgbd_frame" />
+  <joint name="camera_rgbd_joint" type="fixed">
+    <origin xyz="0 0 0" rpy="-${pi/2} 0 -${pi/2}" />
+    <parent link="camera" />
+    <child link="camera_rgbd_frame" />
+  </joint>
   <link name='hokuyo'>
     <inertial>
@@ -157,5 +163,5 @@
       <origin xyz="0 0 0" rpy="0 0 0"/>
       <geometry>
-        <mesh filename="package://udacity_bot/meshes/hokuyo.dae" />
+        <mesh filename="package://slam_bot/meshes/hokuyo.dae" />
       </geometry>
     </visual>
